File: pcbbysid.kicad_sch (KiCad schematic)
At the start: 9 parts, among them Q1 NPN, SW1 SW_Push

Commit message: Add files via upload
Parts:
- added R5: R, Resistor_THT:R_Axial_DIN0207_L6.3mm_D2.5mm_P7.62mm_Horizontal, symbol Device:R
Connections:
- net at BT1.2 (-), R4.2: now also R5.2; no longer Q1.3 (E)
- new net: Q1.3 (E), R5.1
Changed lines of the file:
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@@
-	)
-	(junction
-		(at 105.41 82.55)
-		(diameter 0)
-		(color 0 0 0 0)
 	)
 	(junction
@@
 		(color 0 0 0 0)
 	)
+	(junction
+		(at 105.41 86.36)
+		(diameter 0)
+		(color 0 0 0 0)
+	)
 	(bus_entry
 		(at 59.69 21.59)
@@
 	(wire
 		(pts
-			(xy 105.41 78.74) (xy 105.41 82.55)
+			(xy 105.41 86.36) (xy 113.03 86.36)
 		)
 		(stroke
@@
 	(wire
 		(pts
-			(xy 113.03 82.55) (xy 105.41 82.55)
+			(xy 36.83 86.36) (xy 105.41 86.36)
 		)
 		(stroke
@@
 	(wire
 		(pts
-			(xy 36.83 64.77) (xy 36.83 82.55)
-		)
-		(stroke
-			(width 0)
-			(type default)
-		)
-	)
-	(wire
-		(pts
-			(xy 36.83 82.55) (xy 105.41 82.55)
+			(xy 113.03 86.36) (xy 113.03 82.55)
+		)
+		(stroke
+			(width 0)
+			(type default)
+		)
+	)
+	(wire
+		(pts
+			(xy 36.83 64.77) (xy 36.83 86.36)
 		)
 		(stroke
@@
 					(unit 1)
 				)
+			)
+		)
+	)
+	(symbol
+		(lib_id "Device:R")
+		(at 105.41 82.55 0)
+		(unit 1)
+		(exclude_from_sim no)
+		(in_bom yes)
+		(on_board yes)
+		(dnp no)
+		(fields_autoplaced yes)
+		(property "Reference" "R5"
+			(at 107.95 81.2799 0)
+			(effects
+				(font
+					(size 1.27 1.27)
+				)
+				(justify left)
+			)
+		)
+		(property "Value" "R"
+			(at 107.95 83.8199 0)
+			(effects
+				(font
+					(size 1.27 1.27)
+				)
+				(justify left)
+			)
+		)
+		(property "Footprint" "Resistor_THT:R_Axial_DIN0207_L6.3mm_D2.5mm_P7.62mm_Horizontal"
+			(at 103.632 82.55 90)
+			(effects
+				(font
+					(size 1.27 1.27)
+				)
+				(hide yes)
+			)
+		)
+		(property "Datasheet" "~"
+			(at 105.41 82.55 0)
+			(effects
+				(font
+					(size 1.27 1.27)
+				)
+				(hide yes)
+			)
+		)
+		(property "Description" "Resistor"
+			(at 105.41 82.55 0)
+			(effects
+				(font
+					(size 1.27 1.27)
+				)
+				(hide yes)
+			)
+		)
+		(pin "2"
+		)
+		(pin "1"
+		)
+		(instances
+			(project ""
+				(path "/2228cab5-99d3-4cb0-b1f4-c122c499ff77"
+					(reference "R5")
+					(unit 1)
+				)
